Commit message: hot fix: robot urfd

File: src/caramelo_description/urdf/common_properties.xacro (robot description, xacro)
@@ -1,44 +1,50 @@
 <?xml version="1.0"?>
 <robot xmlns:xacro="http://www.ros.org/wiki/xacro">
+    <!-- Cores padrao do modelo -->
     <material name="blue">
-        <color rgba="0 0 0.5 1" />
+        <color rgba="0 0 0.5 1"/>
     </material>
     <material name="grey">
-        <color rgba="0.5 0.5 0.5 1" />
+        <color rgba="0.5 0.5 0.5 1"/>
     </material>
     <material name="orange">
-        <color rgba="1.0 0.5 0 1" />
+        <color rgba="1.0 0.5 0 1"/>
     </material>
     <material name="yellow">
-        <color rgba="1.0 1.0 0 1" />
+        <color rgba="1.0 1.0 0 1"/>
     </material>
     <material name="darkgray">
         <color rgba="0.3 0.3 0.3 1.0"/>
     </material>
+    <!-- Propriedades centrais do robo -->
+    <xacro:property name="M_PI" value="3.1415926535897931"/>
+    <!-- Inercia de caixa alinhada com os eixos locais -->
     <xacro:macro name="box_inertia" params="m x y z o_xyz o_rpy">
         <inertial>
-            <mass value="${m}" />
-            <origin xyz="${o_xyz}" rpy="${o_rpy}" />
-            <inertia ixx="${(m/12) * (y*y + z*z)}" ixy="0" ixz="0"
-                     iyy="${(m/12) * (x*x + z*z)}" iyz="0"
-                     izz="${(m/12) * (x*x + y*y)}" />
+            <mass value="${m}"/>
+            <origin xyz="${o_xyz}" rpy="${o_rpy}"/>
+            <inertia ixx="${(m/12.0) * (y*y + z*z)}" ixy="0" ixz="0"
+                     iyy="${(m/12.0) * (x*x + z*z)}" iyz="0"
+                     izz="${(m/12.0) * (x*x + y*y)}"/>
         </inertial>
     </xacro:macro>
+    <!-- Inercia de cilindro (eixo principal no eixo Z local) -->
     <xacro:macro name="cylinder_inertia" params="m r l o_xyz o_rpy">
         <inertial>
-            <mass value="${m}" />
-            <origin xyz="${o_xyz}" rpy="${o_rpy}" />
-            <inertia ixx="${(m/12) * (3*r*r + l*l)}" ixy="0" ixz="0"
-                     iyy="${(m/12) * (3*r*r + l*l)}" iyz="0"
-                     izz="${(m/2) * (r*r)}" />
+            <mass value="${m}"/>
+            <origin xyz="${o_xyz}" rpy="${o_rpy}"/>
+            <inertia ixx="${(m/12.0) * (3*r*r + l*l)}" ixy="0" ixz="0"
+                     iyy="${(m/12.0) * (3*r*r + l*l)}" iyz="0"
+                     izz="${(m/2.0) * (r*r)}"/>
         </inertial>
     </xacro:macro>
+    <!-- Inercia de esfera -->
     <xacro:macro name="sphere_inertia" params="m r o_xyz o_rpy">
         <inertial>
-            <mass value="${m}" />
-            <origin xyz="${o_xyz}" rpy="${o_rpy}" />
-            <inertia ixx="${(2/5) * m * r * r}" ixy="0" ixz="0"
-                     iyy="${(2/5) * m * r * r}" iyz="0"
-                     izz="${(2/5) * m * r * r}" />
+            <mass value="${m}"/>
+            <origin xyz="${o_xyz}" rpy="${o_rpy}"/>
+            <inertia ixx="${(2.0/5.0) * m * r * r}" ixy="0" ixz="0"
+                     iyy="${(2.0/5.0) * m * r * r}" iyz="0"
+                     izz="${(2.0/5.0) * m * r * r}"/>
         </inertial>
     </xacro:macro>

File: src/caramelo_description/urdf/lidar_sensor.xacro (robot description, xacro)
@@ -1,5 +1,4 @@
 <?xml version="1.0"?>
 <robot xmlns:xacro="http://www.ros.org/wiki/xacro">
-    <xacro:property name="M_PI" value="3.1415926535897931" />
     <xacro:macro name="lidar_sensor" params="
         prefix:=''
@@ -34,7 +33,4 @@
         visualize:=false
         enable_collision:=false">
-        <xacro:property name="radius" value="${lidar_width/2}" />
-        <xacro:property name="ixx_iyy" value="${(mass/12) * (3 * radius * radius + lidar_height * lidar_height)}" />
-        <xacro:property name="izz" value="${(mass/2) * (radius * radius)}" />
         <link name="${prefix}${frame_id}">
         <visual>
@@ -55,15 +51,10 @@
             </collision>
         </xacro:if>
-        <inertial>
-            <mass value="${mass}" />
-            <origin xyz="${inertial_xyz_offset}" rpy="${inertial_rpy_offset}"/>
-            <inertia
-            ixx="${ixx_iyy}"
-            ixy="0.0"
-            ixz="0.0"
-            iyy="${ixx_iyy}"
-            iyz="0.0"
-            izz="${izz}" />
-        </inertial>
+        <xacro:cylinder_inertia
+            m="${mass}"
+            r="${lidar_width/2}"
+            l="${lidar_height}"
+            o_xyz="${inertial_xyz_offset}"
+            o_rpy="${inertial_rpy_offset}"/>
         </link>
         <joint name="${prefix}${frame_id}_joint" type="fixed">

File: src/caramelo_description/urdf/mecanum_wheel.xacro (robot description, xacro)
@@ -1,46 +1,29 @@
 <?xml version="1.0"?>
 <robot xmlns:xacro="http://www.ros.org/wiki/xacro">
-    <!-- Especificações das rodas mecanum do robô Caramelo -->
-    <xacro:property name="wheel_radius" value="0.05" />
-    <xacro:property name="wheel_width" value="0.069" />
-    <xacro:property name="wheel_mass" value="3.0" />
-    <xacro:property name="wheel_separation" value="0.310" /> <!-- Distância entre as rodas 21 + 3 + 7 -->
-    <xacro:property name="wheel_base" value="0.470" />
+    <!-- Macro de uma roda mecanum -->
     <xacro:macro name="mecanum_wheel" params="prefix side x_reflect y_reflect">
         <link name="${prefix}${side}_wheel_link">
-        <!-- Geometria visual: roda como cilindro -->
-        <visual>
-            <origin xyz="0 0 0" rpy="${pi/2} 0 0"/>
-            <geometry>
-                <cylinder radius="${wheel_radius}" length="${wheel_width}"/>
-            </geometry>
-            <material name="orange">
-                <color rgba="1.0 0.5 0.0 1.0"/>
-            </material>
-        </visual>
-        <!-- Geometria de colisão: cilindro simples para otimização de performance -->
-        <collision>
-            <origin xyz="0 0 0" rpy="${pi/2} 0 0"/>
-            <geometry>
-                <cylinder radius="${wheel_radius}" length="${wheel_width}"/>
-            </geometry>
-        </collision>
-        <!-- Propriedades inerciais baseadas no cilindro -->
-        <inertial>
-            <origin xyz="0 0 0" rpy="0 0 0"/>
-            <mass value="${wheel_mass}"/>
-            <inertia
-                ixx="${(wheel_mass/12.0) * (3*wheel_radius*wheel_radius + wheel_width*wheel_width)}" ixy="0" ixz="0"
-                iyy="${(wheel_mass/2.0) * (wheel_radius*wheel_radius)}" iyz="0"
-                izz="${(wheel_mass/12.0) * (3*wheel_radius*wheel_radius + wheel_width*wheel_width)}"/>
-            </inertial>
+            <visual>
+                <origin xyz="0 0 0" rpy="${M_PI/2} 0 0"/>
+                <geometry>
+                    <cylinder radius="${wheel_radius}" length="${wheel_width}"/>
+                </geometry>
+                <material name="orange"/>
+            </visual>
+            <collision>
+                <origin xyz="0 0 0" rpy="${M_PI/2} 0 0"/>
+                <geometry>
+                    <cylinder radius="${wheel_radius}" length="${wheel_width}"/>
+                </geometry>
+            </collision>
+            <xacro:cylinder_inertia m="${wheel_mass}" r="${wheel_radius}" l="${wheel_width}" o_xyz="0 0 0" o_rpy="${M_PI/2} 0 0"/>
         </link>
-        <!-- Joint da roda: rotação contínua em torno do eixo Y -->
+        <!-- Rotacao continua da roda no eixo Y -->
         <joint name="${prefix}${side}_wheel_joint" type="continuous">
-        <axis xyz="0 1 0"/>
-        <parent link="${prefix}base_link"/>
-        <child link="${prefix}${side}_wheel_link"/>
-        <origin xyz="${x_reflect*(wheel_base/2)} ${y_reflect*(wheel_separation/2)} 0.02" rpy="0 0 0"/>
+            <axis xyz="0 1 0"/>
+            <parent link="${prefix}base_link"/>
+            <child link="${prefix}${side}_wheel_link"/>
+            <origin xyz="${x_reflect*(wheel_base/2)} ${y_reflect*(wheel_separation/2)} 0.02" rpy="0 0 0"/>
         </joint>
-    </xacro:macro> <!-- end mecanum_wheel -->
+    </xacro:macro>
 </robot>

File: src/caramelo_description/urdf/mobile_base.xacro (robot description, xacro)
@@ -1,57 +1,85 @@
 <?xml version="1.0"?>
 <robot xmlns:xacro="http://www.ros.org/wiki/xacro">
-  <!-- Propriedades da base do robô Caramelo -->
-  <xacro:property name="mass" value="22.0"/>
-  <xacro:property name="width_vertical" value="0.550"/>   <!-- Comprimento -->
-  <xacro:property name="depth_vertical" value="0.210"/>   <!-- Largura -->
-  <xacro:property name="width_horizontal" value="0.330"/>   <!-- Comprimento -->
-  <xacro:property name="depth_horizontal" value="0.320"/>   <!-- Largura -->
-  <xacro:property name="height" value="0.105"/>  <!-- Altura -->
-  <xacro:property name="wheel_radius" value="0.05"/>
-  <xacro:macro name="robot_base" params="prefix">
-    <!-- Basefootprint link -->
+    <xacro:include filename="mecanum_wheel.xacro"/>
+    <!-- Parametros especificos do robo Caramelo -->
+    <xacro:property name="base_mass" value="22.0"/>
+    <xacro:property name="base_height" value="0.105"/>
+    <xacro:property name="base_width_vertical" value="0.550"/>
+    <xacro:property name="base_depth_vertical" value="0.210"/>
+    <xacro:property name="base_width_horizontal" value="0.330"/>
+    <xacro:property name="base_depth_horizontal" value="0.320"/>
+    <xacro:property name="wheel_radius" value="0.05"/>
+    <xacro:property name="wheel_width" value="0.069"/>
+    <xacro:property name="wheel_mass" value="3.0"/>
+    <xacro:property name="wheel_separation" value="0.310"/>
+    <xacro:property name="wheel_base" value="0.470"/>
+    <!-- Base completa: footprint + base_link + 4 rodas mecanum -->
+    <xacro:macro name="mobile_base" params="prefix">
     <link name="${prefix}base_footprint"/>
-    <!-- Link da base (base_link agora toca o chão) -->
     <link name="${prefix}base_link">
-      <visual>
-        <origin xyz="0 0 ${height/2.0}" rpy="0 0 0"/>
-        <geometry>
-          <box size="${width_vertical} ${depth_vertical} ${height}"/>
-        </geometry>
-        <material name="darkgray">
-          <color rgba="0.3 0.3 0.3 1.0"/>
-        </material>
-      </visual>
-      <visual>
-        <origin xyz="0 0 ${height/2.0}" rpy="0 0 0"/>
-        <geometry>
-          <box size="${depth_horizontal} ${width_horizontal} ${height}"/>
-        </geometry>
-        <material name="darkgray">
-          <color rgba="0.3 0.3 0.3 1.0"/>
-        </material>
-      </visual>
-      <collision>
-        <origin xyz="0 0 ${height/2.0}" rpy="0 0 0"/>
-        <geometry>
-          <box size="${width_vertical} ${depth_vertical} ${height}"/>
-        </geometry>
-      </collision>
-      <inertial>
-        <mass value="${mass}"/>
-        <origin xyz="0 0 ${height/2.0}" rpy="0 0 0"/>
-        <inertia
-          ixx="${1/12.0 * mass * (height*height + depth_vertical*depth_vertical)}"
-          iyy="${1/12.0 * mass * (width_vertical*width_vertical + depth_vertical*depth_vertical)}"
-          izz="${1/12.0 * mass * (width_vertical*width_vertical + height*height)}"
-          ixy="0.0" ixz="0.0" iyz="0.0"/>
-      </inertial>
+        <!-- Corpo principal em cruz (duas caixas visuais) -->
+        <visual>
+            <origin xyz="0 0 ${base_height/2.0}" rpy="0 0 0"/>
+            <geometry>
+                <box size="${base_width_vertical} ${base_depth_vertical} ${base_height}"/>
+            </geometry>
+            <material name="darkgray"/>
+        </visual>
+        <visual>
+            <origin xyz="0 0 ${base_height/2.0}" rpy="0 0 0"/>
+            <geometry>
+                <box size="${base_depth_horizontal} ${base_width_horizontal} ${base_height}"/>
+            </geometry>
+            <material name="darkgray"/>
+        </visual>
+        <!-- Colisao em cruz para casar com a geometria visual -->
+        <collision>
+            <origin xyz="0 0 ${base_height/2.0}" rpy="0 0 0"/>
+            <geometry>
+                <box size="${base_width_vertical} ${base_depth_vertical} ${base_height}"/>
+            </geometry>
+        </collision>
+        <collision>
+            <origin xyz="0 0 ${base_height/2.0}" rpy="0 0 0"/>
+            <geometry>
+                <box size="${base_depth_horizontal} ${base_width_horizontal} ${base_height}"/>
+            </geometry>
+        </collision>
+        <!-- Inercia aproximada por caixa envolvente da base -->
+        <xacro:box_inertia
+            m="${base_mass}"
+            x="${base_width_vertical}"
+            y="${base_width_horizontal}"
+            z="${base_height}"
+            o_xyz="0 0 ${base_height/2.0}"
+            o_rpy="0 0 0"/>
     </link>
-    <!-- Joint com o footprint (ajustado para as dimensões do Caramelo) -->
+    <!-- Base apoiada nas rodas -->
     <joint name="${prefix}base_joint" type="fixed">
-      <parent link="${prefix}base_footprint"/>
-      <child link="${prefix}base_link"/>
-      <origin xyz="0 0 ${wheel_radius - 0.02}" rpy="0 0 0"/>
+        <parent link="${prefix}base_footprint"/>
+        <child link="${prefix}base_link"/>
+        <origin xyz="0 0 ${wheel_radius - 0.02}" rpy="0 0 0"/>
     </joint>
+    <!-- Quatro rodas mecanum -->
+    <xacro:mecanum_wheel
+        prefix="${prefix}"
+        side="front_left"
+        x_reflect="1"
+        y_reflect="1"/>
+    <xacro:mecanum_wheel
+        prefix="${prefix}"
+        side="front_right"
+        x_reflect="1"
+        y_reflect="-1"/>
+    <xacro:mecanum_wheel
+        prefix="${prefix}"
+        side="back_left"
+        x_reflect="-1"
+        y_reflect="1"/>
+    <xacro:mecanum_wheel
+        prefix="${prefix}"
+        side="back_right"
+        x_reflect="-1"
+        y_reflect="-1"/>
   </xacro:macro>
 </robot>

File: src/caramelo_description/urdf/robot.urdf.xacro (robot description, xacro)
@@ -1,40 +1,15 @@
 <?xml version="1.0"?>
 <robot name="caramelo" xmlns:xacro="http://ros.org/wiki/xacro">
-  <!-- Propriedades -->
-  <xacro:property name="M_PI" value="3.1415926535897931" />
   <!-- Argumentos -->
   <xacro:arg name="robot_name" default="caramelo"/>
   <xacro:arg name="prefix" default=""/>
-  <!-- Inclusões -->
-  <xacro:include filename="common_properties.xacro" />
-  <xacro:include filename="mecanum_wheel.xacro" />
-  <xacro:include filename="lidar_sensor.xacro" />
-  <xacro:include filename="mobile_base.xacro" />
-  <xacro:include filename="mobile_base.ros2_control.xacro" />
-  <!-- Base -->
-  <xacro:robot_base
-    prefix="$(arg prefix)"/>
-  <!-- Rodas mecanum -->
-  <xacro:mecanum_wheel
-    prefix="$(arg prefix)"
-    side="front_left"
-    x_reflect="1"
-    y_reflect="1"/>
-  <xacro:mecanum_wheel
-    prefix="$(arg prefix)"
-    side="front_right"
-    x_reflect="1"
-    y_reflect="-1"/>
-  <xacro:mecanum_wheel
-    prefix="$(arg prefix)"
-    side="back_left"
-    x_reflect="-1"
-    y_reflect="1"/>
-  <xacro:mecanum_wheel
-    prefix="$(arg prefix)"
-    side="back_right"
-    x_reflect="-1"
-    y_reflect="-1"/>
-  <!-- RPLidar S2 - Posicionado na face frontal do robô -->
+  <!-- Includes -->
+  <xacro:include filename="common_properties.xacro"/>
+  <xacro:include filename="lidar_sensor.xacro"/>
+  <xacro:include filename="mobile_base.xacro"/>
+  <xacro:include filename="mobile_base.ros2_control.xacro"/>
+  <!-- Base movel completa (base_link + footprint + 4 rodas) -->
+  <xacro:mobile_base prefix="$(arg prefix)"/>
+  <!-- Sensor lidar -->
   <xacro:lidar_sensor
     prefix="$(arg prefix)"
